File: kicad/pisynth/pisynth.kicad_pcb (KiCad board)
At the start: 2 copper layers, 100 x 100 mm, 52 parts, among them J1 Out Audio, J3 Out Volt, U1 Pico, U2 Volume Pot, U3 MyPotType1, U4 MyPotType1, U5 MyPotType1

Commit message: update
Parts:
- removed C2: C47uf, myFootprints:myCapacitor
- removed OutVoltLed1: LED, myFootprints:myLed
- removed R2: R100om, myFootprints:myResistor
- removed R3: R1.8kom, myFootprints:myResistor
- R1: value R220 -> R1_8kom
- moved U3 17.9 mm to (34.8, 71.0)
- moved U4 17.9 mm to (34.8, 101.0)
- moved U5 16.2 mm to (34.8, 131.0)
- moved U1 15.0 mm to (48.5, 49.0)
- moved G*** 7.57 mm to (80.3, 85.0)
- moved C1 4.01 mm to (120.8, 39.5), turned to 180 degrees
- moved R1 3.20 mm to (127.0, 52.0)
Connections:
- C1 pad 1: Net-(C1-Pad1) -> Net-(U2-Pad3)
- R1 pad 1: Net-(C1-Pad1) -> Net-(U2-Pad3)
- U2 pad 3: Net-(C2-Pad2) -> Net-(U2-Pad3)
Routing:
- net Net-(U2-Pad3): track 0.00 -> 72.7 mm
- net Net-(C1-Pad1): track 50.1 -> 0.00 mm
- net GND: track 16.1 -> 57.5 mm, vias 8 -> 5
- net Net-(C2-Pad2): track 22.7 -> 0.00 mm
- net Net-(H11-Pad1): track 382.4 -> 400.4 mm
- net Net-(Pot2Led1-Pad2): track 71.5 -> 88.6 mm
- net Net-(H3-Pad1): track 124.5 -> 107.7 mm
- net Net-(H8-Pad1): track 96.3 -> 112.8 mm
- net Net-(H4-Pad1): track 151.7 -> 135.8 mm
- net Net-(H2-Pad1): track 174.9 -> 159.4 mm
- net Net-(LFOLed1-Pad2): track 255.9 -> 270.9 mm
- net Net-(H1-Pad1): track 203.0 -> 188.0 mm
- net Net-(R1-Pad2): track 124.8 -> 139.5 mm
- net Net-(H21-Pad1): track 254.4 -> 269.1 mm
- net Net-(H14-Pad1): track 111.4 -> 97.1 mm
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Other:
- board size 100 x 100 mm -> 115.5 x 100 mm
