File: kicad/pisynth/pisynth.kicad_sch (KiCad schematic)
At the start: 51 parts, among them J1 Out Audio, J3 Out Volt, U1 Pico, U2 Volume Pot, U3 MyPotType1, U4 MyPotType1, U5 MyPotType1

Commit message: update
Parts:
- removed C2: C47uf, myFootprints:myCapacitor, symbol Device:C
- removed OutVoltLed1: LED, myFootprints:myLed, symbol Device:LED
- removed R2: R100om, myFootprints:myResistor, symbol Device:R
- removed R3: R1.8kom, myFootprints:myResistor, symbol Device:R
- R1: value R220 -> R1_8kom
Connections:
- net at C1.1, R1.1: now also U2.3
